Commit message: commit

File: arduinobot_ws/src/arduinobot_description/urdf/snake.urdf (robot description, URDF)
Before this commit: robot origins, 7 links, 6 joints
Links:
- link base_link: geometry collision cylinder length=0.6 radius=0.2; visual cylinder length=0.6 radius=0.2
- link connector1: geometry collision sphere radius=0.2; visual sphere radius=0.2
- link connector2: geometry collision sphere radius=0.2; visual sphere radius=0.2
- link connector3: geometry collision sphere radius=0.2; visual sphere radius=0.2
- link link1: geometry collision cylinder length=0.6 radius=0.2; visual cylinder length=0.6 radius=0.2
- link link2: geometry collision cylinder length=0.6 radius=0.2; visual cylinder length=0.6 radius=0.2
- link link3: geometry collision cylinder length=0.6 radius=0.2; visual cylinder length=0.6 radius=0.2
Joints:
- joint base_to_connector: axis (none) -> 0 0 1; limit (none) -> lower=-1.5707 upper=1.5707 effort=1000.0 velocity=0.5; type fixed -> revolute
- joint link1_to_connector2: axis (none) -> 0 0 1; limit (none) -> lower=-1.5707 upper=1.5707 effort=1000.0 velocity=0.5; type fixed -> revolute
- joint link2_to_connector3: axis (none) -> 0 0 1; limit (none) -> lower=-1.5707 upper=1.5707 effort=1000.0 velocity=0.5; type fixed -> revolute
