Commit message: inertia added

File: snake_ws/install/snake_robot_description/share/snake_robot_description/urdf/common_properties.xacro (robot description, xacro)
@@ -2,11 +2,31 @@
 <robot xmlns:xacro="http://ros.org/wiki/xacro">
     <material name="blue">
-        <color rgba="0 0 0.8 1"/>
+        <color rgba="0 0 0.8 0.5"/>
     </material>
     <material name="white">
-        <color rgba="1 1 1 1"/>
+        <color rgba="1 1 1 0.5"/>
     </material>
     <material name="red">
-        <color rgba="0.8 0 0 1"/>
+        <color rgba="0.8 0 0 0.5"/>
     </material>
+    <xacro:macro name="cylinder_inertia" params="m r h xyz rpy" >
+        <inertial>
+            <origin xyz="${xyz}" rpy="${rpy}"/>
+            <mass value="${m}"/>
+            <inertia    ixx="${(m/12) * (3*r*r + h*h)}"  ixy="0"  ixz="0"
+                        iyy="${(m/12) * (3*r*r + h*h)}"  iyz="0"
+                        izz="${(m/2) * (r*r)}"
+            />
+        </inertial>
+    </xacro:macro>
+    <xacro:macro name="sphere_inertia" params="m r xyz rpy" >
+        <inertial>
+            <origin xyz="${xyz}" rpy="${rpy}"/>
+            <mass value="${m}"/>
+            <inertia    ixx="${(2/5) * (m*r*r)}"  ixy="0"  ixz="0"
+                        iyy="${(2/5) * (m*r*r)}"  iyz="0"
+                        izz="${(2/5) * (m*r*r)}"
+            />
+        </inertial>
+    </xacro:macro>
 </robot>

File: snake_ws/install/snake_robot_description/share/snake_robot_description/urdf/components.xacro (robot description, xacro)
@@ -3,19 +3,4 @@
 <xacro:property name="piperdius" value="0.2" />
 <xacro:property name="pipelen" value="0.6" />
-<xacro:macro name="connector_macro" params="postfix">
-    <link name="connector${postfix}">
-        <visual>
-          <geometry>
-            <sphere radius="${piperdius}"/>
-          </geometry>
-          <material name="red"/>
-        </visual>
-        <collision>
-            <geometry>
-                <sphere radius="${piperdius}"/>
-            </geometry>
-          </collision>
-      </link>
-</xacro:macro>
 <xacro:macro name="link_macro" params="name x_origin y_origin z_origin">
     <link name="${name}">
@@ -27,4 +12,5 @@
             <material name="white"/>
         </visual>
+        <xacro:cylinder_inertia  m="1" r="${piperdius}" h="${pipelen}" xyz="${x_origin} ${y_origin} ${z_origin}" rpy="0 ${pi / 2.0} ${pi / 2.0}"/>
         <collision>
             <geometry>
@@ -42,4 +28,21 @@
         <origin xyz="${x_origin} ${y_origin} ${z_origin}"/>
     </joint>
+</xacro:macro>
+<xacro:macro name="connector_macro" params="postfix">
+    <link name="connector${postfix}">
+        <visual>
+          <geometry>
+            <sphere radius="${piperdius}"/>
+          </geometry>
+          <material name="red"/>
+          <origin rpy="0 0 0" xyz="0 0 0"/>
+        </visual>
+        <xacro:sphere_inertia  m="0.5" r="${piperdius}" xyz="0 0 0" rpy="0 0 0"/>
+        <collision>
+            <geometry>
+                <sphere radius="${piperdius}"/>
+            </geometry>
+          </collision>
+      </link>
 </xacro:macro>
 <xacro:macro name="connector_to_link_macro" params="name x_origin y_origin z_origin parent child">

File: snake_ws/src/snake_robot_description/urdf/components_with_collision.xacro (robot description, xacro)
@@ -3,4 +3,19 @@
 <xacro:property name="piperdius" value="0.2" />
 <xacro:property name="pipelen" value="0.6" />
+<xacro:macro name="connector_macro" params="postfix">
+    <link name="connector${postfix}">
+        <visual>
+          <geometry>
+            <sphere radius="${piperdius}"/>
+          </geometry>
+          <material name="red"/>
+        </visual>
+        <collision>
+            <geometry>
+                <sphere radius="${piperdius}"/>
+            </geometry>
+          </collision>
+      </link>
+</xacro:macro>
 <xacro:macro name="link_macro" params="name x_origin y_origin z_origin">
     <link name="${name}">
@@ -12,5 +27,4 @@
             <material name="white"/>
         </visual>
-        <xacro:cylinder_inertia  m="1" r="${piperdius}" h="${pipelen}" xyz="${x_origin} ${y_origin} ${z_origin}" rpy="0 ${pi / 2.0} ${pi / 2.0}"/>
         <collision>
             <geometry>
@@ -28,21 +42,4 @@
         <origin xyz="${x_origin} ${y_origin} ${z_origin}"/>
     </joint>
-</xacro:macro>
-<xacro:macro name="connector_macro" params="postfix">
-    <link name="connector${postfix}">
-        <visual>
-          <geometry>
-            <sphere radius="${piperdius}"/>
-          </geometry>
-          <material name="red"/>
-          <origin rpy="0 0 0" xyz="0 0 0"/>
-        </visual>
-        <xacro:sphere_inertia  m="0.5" r="${piperdius}" xyz="0 0 0" rpy="0 0 0"/>
-        <collision>
-            <geometry>
-                <sphere radius="${piperdius}"/>
-            </geometry>
-          </collision>
-      </link>
 </xacro:macro>
 <xacro:macro name="connector_to_link_macro" params="name x_origin y_origin z_origin parent child">
