Commit message: starting with gazebo colors

File: snake_ws/install/snake_robot_description/share/snake_robot_description/urdf/components.xacro (robot description, xacro)
@@ -12,10 +12,11 @@
             <material name="white"/>
         </visual>
-        <xacro:cylinder_inertia  m="1" r="${piperdius}" h="${pipelen}" xyz="${x_origin} ${y_origin} ${z_origin}" rpy="0 ${pi / 2.0} ${pi / 2.0}"/>
         <collision>
             <geometry>
                 <cylinder length="${pipelen}" radius="${piperdius}"/>
             </geometry>
-          </collision>
+            <origin rpy="0 ${pi / 2.0} ${pi / 2.0}" xyz="${x_origin} ${y_origin} ${z_origin}"/>
+        </collision>
+        <xacro:cylinder_inertia  m="1" r="${piperdius}" h="${pipelen}" xyz="${x_origin} ${y_origin} ${z_origin}" rpy="0 ${pi / 2.0} ${pi / 2.0}"/>
     </link>
 </xacro:macro>
@@ -38,10 +39,11 @@
           <origin rpy="0 0 0" xyz="0 0 0"/>
         </visual>
-        <xacro:sphere_inertia  m="0.5" r="${piperdius}" xyz="0 0 0" rpy="0 0 0"/>
         <collision>
             <geometry>
                 <sphere radius="${piperdius}"/>
             </geometry>
-          </collision>
+            <origin rpy="0 0 0" xyz="0 0 0"/>
+        </collision>
+        <xacro:sphere_inertia  m="0.5" r="${piperdius}" xyz="0 0 0" rpy="0 0 0"/>
       </link>
 </xacro:macro>

File: snake_ws/install/snake_robot_description/share/snake_robot_description/urdf/snake_urdf.xacro (robot description, xacro)
@@ -1,5 +1,6 @@
 <?xml version="1.0"?>
 <robot name="snake robot" xmlns:xacro="http://ros.org/wiki/xacro">
-<xacro:include filename="common_properties.xacro" />
-<xacro:include filename="components.xacro" />
+    <xacro:include filename="snake_common_properties.xacro" />
+    <xacro:include filename="snake_components.xacro" />
+    <xacro:include filename="snake_components_gazebo.xacro" />
 </robot>
