Commit message: camera added in rvia and gazebo

File: snake_ws/install/snake_robot_description/share/snake_robot_description/urdf/snake_common_properties.xacro (robot description, xacro)
@@ -20,4 +20,14 @@
         </inertial>
     </xacro:macro>
+    <xacro:macro name="box_inertia" params="m l w h xyz rpy" >
+        <inertial>
+            <origin xyz="${xyz}" rpy="${rpy}"/>
+            <mass value="${m}"/>
+            <inertia    ixx="${(m/12) * (h*h + l*l)}"  ixy="0"  ixz="0"
+                        iyy="${(m/12) * (w*w + l*l)}"  iyz="0"
+                        izz="${(m/12) * (w*w + h*h)}"
+            />
+        </inertial>
+    </xacro:macro>
     <xacro:macro name="sphere_inertia" params="m r xyz rpy" >
         <inertial>

File: snake_ws/install/snake_robot_description/share/snake_robot_description/urdf/snake_components.xacro (robot description, xacro)
@@ -1,7 +1,7 @@
 <?xml version="1.0"?>
 <robot xmlns:xacro="http://ros.org/wiki/xacro">
-    <xacro:property name="piperdius" value="0.2" />
-    <xacro:property name="pipelen" value="0.6" />
-    <xacro:macro name="link_macro" params="name x_origin y_origin z_origin">
+    <xacro:property name="piperdius" value="0.1" />
+    <xacro:property name="pipelen" value="0.4" />
+    <xacro:macro name="link_macro" params="name x_origin y_origin z_origin color">
         <link name="${name}">
             <visual>
@@ -10,5 +10,5 @@
                 </geometry>
                 <origin rpy="0 ${pi / 2.0} ${pi / 2.0}" xyz="${x_origin} ${y_origin} ${z_origin}"/>
-                <material name="white"/>
+                <material name="${color}"/>
             </visual>
             <collision>
@@ -21,7 +21,16 @@
         </link>
     </xacro:macro>
-    <xacro:macro name="link_to_connector_macro" params="name x_origin y_origin z_origin parent child">
+    <xacro:macro name="link_to_link_Zaxis_macro" params="name x_origin y_origin z_origin parent child">
         <joint name="${name}" type="revolute">
             <axis xyz="0 0 1"/>
+            <limit effort="1000.0" lower="-${pi / 2.0}" upper="${pi / 2.0}" velocity="0.5"/>
+            <parent link="${parent}"/>
+            <child link="${child}"/>
+            <origin xyz="${x_origin} ${y_origin} ${z_origin}"/>
+        </joint>
+    </xacro:macro>
+    <xacro:macro name="link_to_link_Xaxis_macro" params="name x_origin y_origin z_origin parent child">
+        <joint name="${name}" type="revolute">
+            <axis xyz="1 0 0"/>
             <limit effort="1000.0" lower="-${pi / 2.0}" upper="${pi / 2.0}" velocity="0.5"/>
             <parent link="${parent}"/>
@@ -55,16 +64,20 @@
         </joint>
     </xacro:macro>
-    <xacro:link_macro name="base_link" x_origin="0" y_origin="0" z_origin="0.2"/>
-    <xacro:link_to_connector_macro name="base_to_connector" x_origin="0" y_origin="0.5" z_origin="0.2" parent="base_link" child="connector1"/>
-    <xacro:connector_macro postfix="1" />
-    <xacro:connector_to_link_macro name="connector1_to_link1" x_origin="0" y_origin="0.2" z_origin="0" parent="connector1" child="link1"/>
-    <xacro:link_macro name="link1" x_origin="0" y_origin="0.3" z_origin="0"/>
-    <xacro:link_to_connector_macro name="link1_to_connector2" x_origin="0" y_origin="0.8" z_origin="0" parent="link1" child="connector2"/>
-    <xacro:connector_macro postfix="2" />
-    <xacro:connector_to_link_macro name="connector2_to_link2" x_origin="0" y_origin="0.2" z_origin="0" parent="connector2" child="link2"/>
-    <xacro:link_macro name="link2" x_origin="0" y_origin="0.3" z_origin="0"/>
-    <xacro:link_to_connector_macro name="link2_to_connector3" x_origin="0" y_origin="0.8" z_origin="0" parent="link2" child="connector3"/>
-    <xacro:connector_macro postfix="3" />
-    <xacro:connector_to_link_macro name="connector3_to_link3" x_origin="0" y_origin="0.2" z_origin="0" parent="connector3" child="link3"/>
-    <xacro:link_macro name="link3" x_origin="0" y_origin="0.3" z_origin="0"/>
+    <xacro:link_macro name="base_link" x_origin="0" y_origin="0" z_origin="${piperdius}" color="red"/>
+    <xacro:link_to_link_Zaxis_macro name="base_to_link1_Zaxis" x_origin="0" y_origin="${pipelen / 2}" z_origin="${piperdius}" parent="base_link" child="link1"/>
+    <xacro:link_macro name="link1" x_origin="0" y_origin="${pipelen / 2}" z_origin="0" color="blue"/>
+    <xacro:link_to_link_Xaxis_macro name="link1_to_link2_Xaxis" x_origin="0" y_origin="${pipelen}" z_origin="0" parent="link1" child="link2"/>
+    <xacro:link_macro name="link2" x_origin="0" y_origin="${pipelen / 2}" z_origin="0" color="red"/>
+    <xacro:link_to_link_Zaxis_macro name="link2_to_link3_Zaxis" x_origin="0" y_origin="${pipelen}" z_origin="0" parent="link2" child="link3"/>
+    <xacro:link_macro name="link3" x_origin="0" y_origin="${pipelen / 2}" z_origin="0" color="blue"/>
+    <xacro:link_to_link_Xaxis_macro name="link3_to_link4_Xaxis" x_origin="0" y_origin="${pipelen}" z_origin="0" parent="link3" child="link4"/>
+    <xacro:link_macro name="link4" x_origin="0" y_origin="${pipelen / 2}" z_origin="0" color="red"/>
+    <xacro:link_to_link_Zaxis_macro name="link4_to_link5_Zaxis" x_origin="0" y_origin="${pipelen}" z_origin="0" parent="link4" child="link5"/>
+    <xacro:link_macro name="link5" x_origin="0" y_origin="${pipelen / 2}" z_origin="0" color="blue"/>
+    <xacro:link_to_link_Xaxis_macro name="link5_to_link6_Xaxis" x_origin="0" y_origin="${pipelen}" z_origin="0" parent="link5" child="link6"/>
+    <xacro:link_macro name="link6" x_origin="0" y_origin="${pipelen / 2}" z_origin="0" color="red"/>
+    <xacro:link_to_link_Zaxis_macro name="link6_to_link7_Zaxis" x_origin="0" y_origin="${pipelen}" z_origin="0" parent="link6" child="link7"/>
+    <xacro:link_macro name="link7" x_origin="0" y_origin="${pipelen / 2}" z_origin="0" color="blue"/>
+    <xacro:link_to_link_Xaxis_macro name="link7_to_link8_Xaxis" x_origin="0" y_origin="${pipelen}" z_origin="0" parent="link7" child="link8"/>
+    <xacro:link_macro name="link8" x_origin="0" y_origin="${pipelen / 2}" z_origin="0" color="red"/>
 </robot>

File: snake_ws/install/snake_robot_description/share/snake_robot_description/urdf/snake_components_gazebo.xacro (robot description, xacro)
@@ -2,16 +2,10 @@
 <robot xmlns:xacro="http://ros.org/wiki/xacro">
     <gazebo reference="base_link">
-        <material>Gazebo/Blue</material>
+        <material>Gazebo/Red</material>
     </gazebo>
     <gazebo reference="link1">
         <material>Gazebo/Blue</material>
     </gazebo>
-    <gazebo reference="connector1">
-        <material>Gazebo/Red</material>
-    </gazebo>
     <gazebo reference="link2">
-        <material>Gazebo/Blue</material>
-    </gazebo>
-    <gazebo reference="connector2">
         <material>Gazebo/Red</material>
     </gazebo>
@@ -19,9 +13,18 @@
         <material>Gazebo/Blue</material>
     </gazebo>
-    <gazebo reference="connector3">
+    <gazebo reference="link4">
         <material>Gazebo/Red</material>
     </gazebo>
-    <gazebo reference="base_link">
+    <gazebo reference="link5">
         <material>Gazebo/Blue</material>
     </gazebo>
+    <gazebo reference="link6">
+        <material>Gazebo/Red</material>
+    </gazebo>
+    <gazebo reference="link7">
+        <material>Gazebo/Blue</material>
+    </gazebo>
+    <gazebo reference="link8">
+        <material>Gazebo/Red</material>
+    </gazebo>
 </robot>

File: snake_ws/install/snake_robot_description/share/snake_robot_description/urdf/snake_urdf.xacro (robot description, xacro)
@@ -4,3 +4,4 @@
     <xacro:include filename="snake_components.xacro" />
     <xacro:include filename="snake_components_gazebo.xacro" />
+    <xacro:include filename="snake_camera.xacro" />
 </robot>

File: snake_ws/src/snake_robot_description/urdf/snake_components_gazebo.xacro (robot description, xacro)
@@ -2,16 +2,10 @@
 <robot xmlns:xacro="http://ros.org/wiki/xacro">
     <gazebo reference="base_link">
-        <material>Gazebo/Blue</material>
+        <material>Gazebo/Red</material>
     </gazebo>
     <gazebo reference="link1">
         <material>Gazebo/Blue</material>
     </gazebo>
-    <gazebo reference="connector1">
-        <material>Gazebo/Red</material>
-    </gazebo>
     <gazebo reference="link2">
-        <material>Gazebo/Blue</material>
-    </gazebo>
-    <gazebo reference="connector2">
         <material>Gazebo/Red</material>
     </gazebo>
@@ -19,11 +13,18 @@
         <material>Gazebo/Blue</material>
     </gazebo>
-    <gazebo reference="connector3">
+    <gazebo reference="link4">
         <material>Gazebo/Red</material>
     </gazebo>
-    <gazebo reference="base_link">
+    <gazebo reference="link5">
         <material>Gazebo/Blue</material>
     </gazebo>
-    <gazebo>
+    <gazebo reference="link6">
+        <material>Gazebo/Red</material>
+    </gazebo>
+    <gazebo reference="link7">
+        <material>Gazebo/Blue</material>
+    </gazebo>
+    <gazebo reference="link8">
+        <material>Gazebo/Red</material>
     </gazebo>
 </robot>

Commit message: plugins gazebo_ros_joint_state_publisher and gazebo_ros_joint_pose_trajectory added, to observe and set the joint states

File: snake_ws/install/snake_robot_description/share/snake_robot_description/urdf/snake_common_properties.xacro (robot description, xacro)
@@ -1,4 +1,5 @@
 <?xml version="1.0"?>
 <robot xmlns:xacro="http://ros.org/wiki/xacro">
+    <!-- Define a color materials with RGBA color values -->
     <material name="blue">
         <color rgba="0 0 0.8 0.5"/>
@@ -10,8 +11,10 @@
         <color rgba="0.8 0 0 0.5"/>
     </material>
+    <!-- Define a macro for creating inertia properties for a cylinder -->
     <xacro:macro name="cylinder_inertia" params="m r h xyz rpy" >
         <inertial>
             <origin xyz="${xyz}" rpy="${rpy}"/>
             <mass value="${m}"/>
+            <!-- Calculate and set the inertia tensor values, formula source https://en.wikipedia.org/wiki/List_of_moments_of_inertia -->
             <inertia    ixx="${(m/12) * (3*r*r + h*h)}"  ixy="0"  ixz="0"
                         iyy="${(m/12) * (3*r*r + h*h)}"  iyz="0"
@@ -20,8 +23,10 @@
         </inertial>
     </xacro:macro>
+    <!-- Define a macro for creating inertia properties for a box -->
     <xacro:macro name="box_inertia" params="m l w h xyz rpy" >
         <inertial>
             <origin xyz="${xyz}" rpy="${rpy}"/>
             <mass value="${m}"/>
+            <!-- Calculate and set the inertia tensor values, formula source https://en.wikipedia.org/wiki/List_of_moments_of_inertia -->
             <inertia    ixx="${(m/12) * (h*h + l*l)}"  ixy="0"  ixz="0"
                         iyy="${(m/12) * (w*w + l*l)}"  iyz="0"
@@ -30,8 +35,10 @@
         </inertial>
     </xacro:macro>
+    <!-- Define a macro for creating inertia properties for a sphere -->
     <xacro:macro name="sphere_inertia" params="m r xyz rpy" >
         <inertial>
             <origin xyz="${xyz}" rpy="${rpy}"/>
             <mass value="${m}"/>
+            <!-- Calculate and set the inertia tensor values, formula source https://en.wikipedia.org/wiki/List_of_moments_of_inertia -->
             <inertia    ixx="${(2/5) * (m*r*r)}"  ixy="0"  ixz="0"
                         iyy="${(2/5) * (m*r*r)}"  iyz="0"

File: snake_ws/install/snake_robot_description/share/snake_robot_description/urdf/snake_components.xacro (robot description, xacro)
@@ -1,6 +1,8 @@
 <?xml version="1.0"?>
 <robot xmlns:xacro="http://ros.org/wiki/xacro">
+    <!-- Define variables for reuse -->
     <xacro:property name="piperdius" value="0.1" />
     <xacro:property name="pipelen" value="0.4" />
+    <!-- Define a macro to create a link with visual, collision, and inertia properties -->
     <xacro:macro name="link_macro" params="name x_origin y_origin z_origin color">
         <link name="${name}">
@@ -12,4 +14,5 @@
                 <material name="${color}"/>
             </visual>
+            <!-- Collision properties of the link -->
             <collision>
                 <geometry>
@@ -18,7 +21,9 @@
                 <origin rpy="0 ${pi / 2.0} ${pi / 2.0}" xyz="${x_origin} ${y_origin} ${z_origin}"/>
             </collision>
+            <!-- Inertia properties of the link -->
             <xacro:cylinder_inertia  m="1" r="${piperdius}" h="${pipelen}" xyz="${x_origin} ${y_origin} ${z_origin}" rpy="0 ${pi / 2.0} ${pi / 2.0}"/>
         </link>
     </xacro:macro>
+    <!-- Define a macro to create a revolute joint along the Z-axis between two links -->
     <xacro:macro name="link_to_link_Zaxis_macro" params="name x_origin y_origin z_origin parent child">
         <joint name="${name}" type="revolute">
@@ -28,6 +33,8 @@
             <child link="${child}"/>
             <origin xyz="${x_origin} ${y_origin} ${z_origin}"/>
+            <dynamics friction="0.05" damping="0.1" />
         </joint>
     </xacro:macro>
+    <!-- Define a macro to create a revolute joint along the X-axis between two links -->
     <xacro:macro name="link_to_link_Xaxis_macro" params="name x_origin y_origin z_origin parent child">
         <joint name="${name}" type="revolute">
@@ -37,32 +44,11 @@
             <child link="${child}"/>
             <origin xyz="${x_origin} ${y_origin} ${z_origin}"/>
+            <!--this needs to be investigated, it is adding friction etc-->
+            <dynamics friction="0.05" damping="0.1" />
         </joint>
     </xacro:macro>
-    <xacro:macro name="connector_macro" params="postfix">
-        <link name="connector${postfix}">
-            <visual>
-            <geometry>
-                <sphere radius="${piperdius}"/>
-            </geometry>
-            <material name="red"/>
-            <origin rpy="0 0 0" xyz="0 0 0"/>
-            </visual>
-            <collision>
-                <geometry>
-                    <sphere radius="${piperdius}"/>
-                </geometry>
-                <origin rpy="0 0 0" xyz="0 0 0"/>
-            </collision>
-            <xacro:sphere_inertia  m="0.5" r="${piperdius}" xyz="0 0 0" rpy="0 0 0"/>
-        </link>
-    </xacro:macro>
-    <xacro:macro name="connector_to_link_macro" params="name x_origin y_origin z_origin parent child">
-        <joint name="${name}" type="fixed">
-            <parent link="${parent}"/>
-            <child link="${child}"/>
-            <origin xyz="${x_origin} ${y_origin} ${z_origin}"/>
-        </joint>
-    </xacro:macro>
+    <!-- Create the base link with red color -->
     <xacro:link_macro name="base_link" x_origin="0" y_origin="0" z_origin="${piperdius}" color="red"/>
+    <!-- Create links, joints, and set their positions and colors -->
     <xacro:link_to_link_Zaxis_macro name="base_to_link1_Zaxis" x_origin="0" y_origin="${pipelen / 2}" z_origin="${piperdius}" parent="base_link" child="link1"/>
     <xacro:link_macro name="link1" x_origin="0" y_origin="${pipelen / 2}" z_origin="0" color="blue"/>

File: snake_ws/install/snake_robot_description/share/snake_robot_description/urdf/snake_components_gazebo.xacro (robot description, xacro)
@@ -28,3 +28,25 @@
         <material>Gazebo/Red</material>
     </gazebo>
+    <gazebo>
+        <!-- Plugin introduced from https://github.com/ros-simulation/gazebo_ros_pkgs/blob/ros2/gazebo_plugins/include/gazebo_plugins/gazebo_ros_joint_state_publisher.hpp -->
+        <plugin name="gazebo_ros_joint_state_publisher" filename="libgazebo_ros_joint_state_publisher.so">
+            <!-- Update rate in Hertz -->
+            <update_rate>10</update_rate>
+            <!-- Name of joints in the model whose states will be published. -->
+            <joint_name>base_to_link1_Zaxis</joint_name>
+            <joint_name>link1_to_link2_Xaxis</joint_name>
+            <joint_name>link2_to_link3_Zaxis</joint_name>
+            <joint_name>link3_to_link4_Xaxis</joint_name>
+            <joint_name>link4_to_link5_Zaxis</joint_name>
+            <joint_name>link5_to_link6_Xaxis</joint_name>
+            <joint_name>link6_to_link7_Zaxis</joint_name>
+            <joint_name>link7_to_link8_Xaxis</joint_name>
+        </plugin>
+    </gazebo>
+    <gazebo>
+        <plugin name="gazebo_ros_joint_pose_trajectory" filename="libgazebo_ros_joint_pose_trajectory.so">
+            <!-- Update rate in Hz -->
+            <update_rate>2</update_rate>
+        </plugin>
+    </gazebo>
 </robot>

File: snake_ws/src/snake_robot_description/urdf/snake_camera.xacro (robot description, xacro)
@@ -4,4 +4,5 @@
     <xacro:property name="camera_width" value="0.02" />
     <xacro:property name="camera_height" value="0.05" />
+    <!-- link to hold camera -->
     <link name="camera_link">
         <visual>
@@ -21,6 +22,8 @@
         <parent link="base_link" />
         <child link="camera_link" />
+        <!-- the RPY is NOT 000 to make sure camera does not see inside ground but is over the surface -->
         <origin xyz="0 -${(pipelen + camera_width) / 2} ${piperdius}" rpy="0 -${pi / 16.0} -${pi / 2.0}" />
     </joint>
+    <!-- camera plugin for gazebo -->
     <gazebo reference="camera_link">
         <material>Gazebo/Red</material>

File: snake_ws/src/snake_robot_description/urdf/snake_components_gazebo.xacro (robot description, xacro)
@@ -28,3 +28,27 @@
         <material>Gazebo/Red</material>
     </gazebo>
+    <!-- Plugin introduced from https://github.com/ros-simulation/gazebo_ros_pkgs/blob/ros2/gazebo_plugins/include/gazebo_plugins/gazebo_ros_joint_state_publisher.hpp -->
+    <gazebo>
+        <!-- plugin to publish the states of the robot joints to generate TF -->
+        <plugin name="gazebo_ros_joint_state_publisher" filename="libgazebo_ros_joint_state_publisher.so">
+            <!-- Update rate in Hertz -->
+            <update_rate>10</update_rate>
+            <!-- Name of joints in the model whose states will be published. -->
+            <joint_name>base_to_link1_Zaxis</joint_name>
+            <joint_name>link1_to_link2_Xaxis</joint_name>
+            <joint_name>link2_to_link3_Zaxis</joint_name>
+            <joint_name>link3_to_link4_Xaxis</joint_name>
+            <joint_name>link4_to_link5_Zaxis</joint_name>
+            <joint_name>link5_to_link6_Xaxis</joint_name>
+            <joint_name>link6_to_link7_Zaxis</joint_name>
+            <joint_name>link7_to_link8_Xaxis</joint_name>
+        </plugin>
+    </gazebo>
+    <gazebo>
+        <!-- plugin to set the states of the robot joints -->
+        <plugin name="gazebo_ros_joint_pose_trajectory" filename="libgazebo_ros_joint_pose_trajectory.so">
+            <!-- Update rate in Hz -->
+            <update_rate>2</update_rate>
+        </plugin>
+    </gazebo>
 </robot>
