Commit message: pending addin for revolute join in gazebo

File: snake_ws/install/snake_robot_description/share/snake_robot_description/urdf/snake_components_gazebo.xacro (robot description, xacro)
@@ -4,3 +4,24 @@
         <material>Gazebo/Blue</material>
     </gazebo>
+    <gazebo reference="link1">
+        <material>Gazebo/Blue</material>
+    </gazebo>
+    <gazebo reference="connector1">
+        <material>Gazebo/Red</material>
+    </gazebo>
+    <gazebo reference="link2">
+        <material>Gazebo/Blue</material>
+    </gazebo>
+    <gazebo reference="connector2">
+        <material>Gazebo/Red</material>
+    </gazebo>
+    <gazebo reference="link3">
+        <material>Gazebo/Blue</material>
+    </gazebo>
+    <gazebo reference="connector3">
+        <material>Gazebo/Red</material>
+    </gazebo>
+    <gazebo reference="base_link">
+        <material>Gazebo/Blue</material>
+    </gazebo>
 </robot>

File: snake_ws/src/snake_robot_description/urdf/snake_components_gazebo.xacro (robot description, xacro)
@@ -4,3 +4,26 @@
         <material>Gazebo/Blue</material>
     </gazebo>
+    <gazebo reference="link1">
+        <material>Gazebo/Blue</material>
+    </gazebo>
+    <gazebo reference="connector1">
+        <material>Gazebo/Red</material>
+    </gazebo>
+    <gazebo reference="link2">
+        <material>Gazebo/Blue</material>
+    </gazebo>
+    <gazebo reference="connector2">
+        <material>Gazebo/Red</material>
+    </gazebo>
+    <gazebo reference="link3">
+        <material>Gazebo/Blue</material>
+    </gazebo>
+    <gazebo reference="connector3">
+        <material>Gazebo/Red</material>
+    </gazebo>
+    <gazebo reference="base_link">
+        <material>Gazebo/Blue</material>
+    </gazebo>
+    <gazebo>
+    </gazebo>
 </robot>

Commit message: commit changes , still not working

File: snake_ws/install/snake_robot_description/share/snake_robot_description/urdf/snake_components_gazebo.xacro (robot description, xacro)
@@ -59,17 +59,4 @@
     <xacro:gazebo_link_reference_macro link_name="${link7}" gazebo_color_name="Gazebo/Blue"/>
     <xacro:gazebo_link_reference_macro link_name="${link8}" gazebo_color_name="Gazebo/Red"/>
-    <ros2_control name="GazeboSystem" type="system">
-    	<hardware>
-            <plugin>gazebo_ros2_control/GazeboSystem</plugin>
-    	</hardware>
-        <xacro:ros_control_joint_macro joint_name="${base_to_link1_Zaxis}"/>
-        <xacro:ros_control_joint_macro joint_name="${link1_to_link2_Xaxis}"/>
-        <xacro:ros_control_joint_macro joint_name="${link2_to_link3_Zaxis}"/>
-        <xacro:ros_control_joint_macro joint_name="${link3_to_link4_Xaxis}"/>
-        <xacro:ros_control_joint_macro joint_name="${link4_to_link5_Zaxis}"/>
-        <xacro:ros_control_joint_macro joint_name="${link5_to_link6_Xaxis}"/>
-        <xacro:ros_control_joint_macro joint_name="${link6_to_link7_Zaxis}"/>
-        <xacro:ros_control_joint_macro joint_name="${link7_to_link8_Xaxis}"/>
-    </ros2_control>
     <gazebo>
         <plugin name="gazebo_ros2_control" filename="libgazebo_ros2_control.so">

File: snake_ws/src/snake_robot_description/urdf/scratch.xacro (robot description, xacro)
@@ -44,5 +44,5 @@
     <xacro:macro name="gazebo_link_reference_macro" params="link_name gazebo_color_name">
         <gazebo reference="${link_name}">
-            <material>"${gazebo_color_name}"</material>
+            <material>${gazebo_color_name}</material>
             <mu1>0.01</mu1>
             <mu2>0.05</mu2>
