Commit message: failsafe commit

File: snake_ws/install/snake_robot_description/share/snake_robot_description/urdf/snake_camera.xacro (robot description, xacro)
@@ -4,6 +4,10 @@
     <xacro:property name="camera_width" value="0.02" />
     <xacro:property name="camera_height" value="0.05" />
+    <xacro:property name="camera_link" value="camera_link" />
+    <xacro:property name="camera_joint" value="link8_camera_joint" />
+    <xacro:property name="camera_sensor" value="camera_sensor" />
+    <xacro:property name="camera_controller" value="camera_controller" />
     <!-- link to hold camera -->
-    <link name="camera_link">
+    <link name="${camera_link}">
         <visual>
             <geometry>
@@ -19,18 +23,18 @@
         <xacro:box_inertia m="0.1" l="${camera_length}" w="${camera_width}" h="${camera_height}" xyz="0 0 0" rpy="0 0 0" />
     </link>
-    <joint name="base_camera_joint" type="fixed">
-        <parent link="base_link" />
-        <child link="camera_link" />
+    <joint name="${camera_joint}" type="fixed">
+        <parent link="${link8}" />
+        <child link="${camera_link}" />
         <!-- the RPY is NOT 000 to make sure camera does not see inside ground but is over the surface -->
-        <origin xyz="0 -${(pipelen + camera_width) / 2} ${piperdius}" rpy="0 -${pi / 16.0} -${pi / 2.0}" />
+        <origin xyz="0 ${(pipelen + camera_width)} 0" rpy="0 -${pi / 17.0} ${pi / 2.0}" />
     </joint>
     <!-- camera plugin for gazebo -->
-    <gazebo reference="camera_link">
+    <gazebo reference="${camera_link}">
         <material>Gazebo/Red</material>
-        <sensor name="camera_sensor" type="camera">
+        <sensor name="${camera_sensor}" type="camera">
             <pose>0 0 0 0 0 0</pose>
             <visualize>true</visualize>
             <update_rate>10.0</update_rate>
-            <plugin name="camera_controller" filename="libgazebo_ros_camera.so">
+            <plugin name="${camera_controller}" filename="libgazebo_ros_camera.so">
                 <frame_name>camera_link</frame_name>
             </plugin>

File: snake_ws/install/snake_robot_description/share/snake_robot_description/urdf/snake_components.xacro (robot description, xacro)
@@ -4,4 +4,23 @@
     <xacro:property name="piperdius" value="0.1" />
     <xacro:property name="pipelen" value="0.4" />
+    <!-- Property to define link names -->
+    <xacro:property name="base_link" value="base_link" />
+    <xacro:property name="link1" value="link1" />
+    <xacro:property name="link2" value="link2" />
+    <xacro:property name="link3" value="link3" />
+    <xacro:property name="link4" value="link4" />
+    <xacro:property name="link5" value="link5" />
+    <xacro:property name="link6" value="link6" />
+    <xacro:property name="link7" value="link7" />
+    <xacro:property name="link8" value="link8" />
+    <!-- Property to define joint names -->
+    <xacro:property name="base_to_link1_Zaxis" value="base_to_link1_Zaxis" />
+    <xacro:property name="link1_to_link2_Xaxis" value="link1_to_link2_Xaxis" />
+    <xacro:property name="link2_to_link3_Zaxis" value="link2_to_link3_Zaxis" />
+    <xacro:property name="link3_to_link4_Xaxis" value="link3_to_link4_Xaxis" />
+    <xacro:property name="link4_to_link5_Zaxis" value="link4_to_link5_Zaxis" />
+    <xacro:property name="link5_to_link6_Xaxis" value="link5_to_link6_Xaxis" />
+    <xacro:property name="link6_to_link7_Zaxis" value="link6_to_link7_Zaxis" />
+    <xacro:property name="link7_to_link8_Xaxis" value="link7_to_link8_Xaxis" />
     <!-- Define a macro to create a link with visual, collision, and inertia properties -->
     <xacro:macro name="link_macro" params="name x_origin y_origin z_origin color">
@@ -26,5 +45,5 @@
     </xacro:macro>
     <!-- Define a macro to create a revolute joint along the Z-axis between two links -->
-    <xacro:macro name="link_to_link_Zaxis_macro" params="name x_origin y_origin z_origin parent child">
+    <xacro:macro name="link_to_link_Zaxis_joint_macro" params="name x_origin y_origin z_origin parent child">
         <joint name="${name}" type="revolute">
             <axis xyz="0 0 1"/>
@@ -37,5 +56,5 @@
     </xacro:macro>
     <!-- Define a macro to create a revolute joint along the X-axis between two links -->
-    <xacro:macro name="link_to_link_Xaxis_macro" params="name x_origin y_origin z_origin parent child">
+    <xacro:macro name="link_to_link_Xaxis_joint_macro" params="name x_origin y_origin z_origin parent child">
         <joint name="${name}" type="revolute">
             <axis xyz="1 0 0"/>
@@ -49,21 +68,21 @@
     </xacro:macro>
     <!-- Create the base link with red color -->
-    <xacro:link_macro name="base_link" x_origin="0" y_origin="0" z_origin="${piperdius}" color="red"/>
+    <xacro:link_macro name="${base_link}" x_origin="0" y_origin="0" z_origin="${piperdius}" color="red"/>
     <!-- Create links, joints, and set their positions and colors -->
-    <xacro:link_to_link_Zaxis_macro name="base_to_link1_Zaxis" x_origin="0" y_origin="${pipelen / 2}" z_origin="${piperdius}" parent="base_link" child="link1"/>
-    <xacro:link_macro name="link1" x_origin="0" y_origin="${pipelen / 2}" z_origin="0" color="blue"/>
-    <xacro:link_to_link_Xaxis_macro name="link1_to_link2_Xaxis" x_origin="0" y_origin="${pipelen}" z_origin="0" parent="link1" child="link2"/>
-    <xacro:link_macro name="link2" x_origin="0" y_origin="${pipelen / 2}" z_origin="0" color="red"/>
-    <xacro:link_to_link_Zaxis_macro name="link2_to_link3_Zaxis" x_origin="0" y_origin="${pipelen}" z_origin="0" parent="link2" child="link3"/>
-    <xacro:link_macro name="link3" x_origin="0" y_origin="${pipelen / 2}" z_origin="0" color="blue"/>
-    <xacro:link_to_link_Xaxis_macro name="link3_to_link4_Xaxis" x_origin="0" y_origin="${pipelen}" z_origin="0" parent="link3" child="link4"/>
-    <xacro:link_macro name="link4" x_origin="0" y_origin="${pipelen / 2}" z_origin="0" color="red"/>
-    <xacro:link_to_link_Zaxis_macro name="link4_to_link5_Zaxis" x_origin="0" y_origin="${pipelen}" z_origin="0" parent="link4" child="link5"/>
-    <xacro:link_macro name="link5" x_origin="0" y_origin="${pipelen / 2}" z_origin="0" color="blue"/>
-    <xacro:link_to_link_Xaxis_macro name="link5_to_link6_Xaxis" x_origin="0" y_origin="${pipelen}" z_origin="0" parent="link5" child="link6"/>
-    <xacro:link_macro name="link6" x_origin="0" y_origin="${pipelen / 2}" z_origin="0" color="red"/>
-    <xacro:link_to_link_Zaxis_macro name="link6_to_link7_Zaxis" x_origin="0" y_origin="${pipelen}" z_origin="0" parent="link6" child="link7"/>
-    <xacro:link_macro name="link7" x_origin="0" y_origin="${pipelen / 2}" z_origin="0" color="blue"/>
-    <xacro:link_to_link_Xaxis_macro name="link7_to_link8_Xaxis" x_origin="0" y_origin="${pipelen}" z_origin="0" parent="link7" child="link8"/>
-    <xacro:link_macro name="link8" x_origin="0" y_origin="${pipelen / 2}" z_origin="0" color="red"/>
+    <xacro:link_to_link_Zaxis_joint_macro name="${base_to_link1_Zaxis}" x_origin="0" y_origin="${pipelen / 2}" z_origin="${piperdius}" parent="${base_link}" child="${link1}"/>
+    <xacro:link_macro name="${link1}" x_origin="0" y_origin="${pipelen / 2}" z_origin="0" color="blue"/>
+    <xacro:link_to_link_Xaxis_joint_macro name="${link1_to_link2_Xaxis}" x_origin="0" y_origin="${pipelen}" z_origin="0" parent="${link1}" child="${link2}"/>
+    <xacro:link_macro name="${link2}" x_origin="0" y_origin="${pipelen / 2}" z_origin="0" color="red"/>
+    <xacro:link_to_link_Zaxis_joint_macro name="${link2_to_link3_Zaxis}" x_origin="0" y_origin="${pipelen}" z_origin="0" parent="${link2}" child="${link3}"/>
+    <xacro:link_macro name="${link3}" x_origin="0" y_origin="${pipelen / 2}" z_origin="0" color="blue"/>
+    <xacro:link_to_link_Xaxis_joint_macro name="${link3_to_link4_Xaxis}" x_origin="0" y_origin="${pipelen}" z_origin="0" parent="${link3}" child="${link4}"/>
+    <xacro:link_macro name="${link4}" x_origin="0" y_origin="${pipelen / 2}" z_origin="0" color="red"/>
+    <xacro:link_to_link_Zaxis_joint_macro name="${link4_to_link5_Zaxis}" x_origin="0" y_origin="${pipelen}" z_origin="0" parent="${link4}" child="${link5}"/>
+    <xacro:link_macro name="${link5}" x_origin="0" y_origin="${pipelen / 2}" z_origin="0" color="blue"/>
+    <xacro:link_to_link_Xaxis_joint_macro name="${link5_to_link6_Xaxis}" x_origin="0" y_origin="${pipelen}" z_origin="0" parent="${link5}" child="${link6}"/>
+    <xacro:link_macro name="${link6}" x_origin="0" y_origin="${pipelen / 2}" z_origin="0" color="red"/>
+    <xacro:link_to_link_Zaxis_joint_macro name="${link6_to_link7_Zaxis}" x_origin="0" y_origin="${pipelen}" z_origin="0" parent="${link6}" child="${link7}"/>
+    <xacro:link_macro name="${link7}" x_origin="0" y_origin="${pipelen / 2}" z_origin="0" color="blue"/>
+    <xacro:link_to_link_Xaxis_joint_macro name="${link7_to_link8_Xaxis}" x_origin="0" y_origin="${pipelen}" z_origin="0" parent="${link7}" child="${link8}"/>
+    <xacro:link_macro name="${link8}" x_origin="0" y_origin="${pipelen / 2}" z_origin="0" color="red"/>
 </robot>

File: snake_ws/install/snake_robot_description/share/snake_robot_description/urdf/snake_components_gazebo.xacro (robot description, xacro)
@@ -1,54 +1,88 @@
 <?xml version="1.0"?>
 <robot xmlns:xacro="http://ros.org/wiki/xacro">
-    <gazebo reference="base_link">
-        <material>Gazebo/Red</material>
-    </gazebo>
-    <gazebo reference="link1">
-        <material>Gazebo/Blue</material>
-    </gazebo>
-    <gazebo reference="link2">
-        <material>Gazebo/Red</material>
-    </gazebo>
-    <gazebo reference="link3">
-        <material>Gazebo/Blue</material>
-    </gazebo>
-    <gazebo reference="link4">
-        <material>Gazebo/Red</material>
-    </gazebo>
-    <gazebo reference="link5">
-        <material>Gazebo/Blue</material>
-    </gazebo>
-    <gazebo reference="link6">
-        <material>Gazebo/Red</material>
-    </gazebo>
-    <gazebo reference="link7">
-        <material>Gazebo/Blue</material>
-    </gazebo>
-    <gazebo reference="link8">
-        <material>Gazebo/Red</material>
-    </gazebo>
-    <!-- Plugin introduced from https://github.com/ros-simulation/gazebo_ros_pkgs/blob/ros2/gazebo_plugins/include/gazebo_plugins/gazebo_ros_joint_state_publisher.hpp -->
+    <xacro:property name="base_to_link1_tran" value="base_to_link1_tran" />
+    <xacro:property name="link1_to_link2_tran" value="link1_to_link2_tran" />
+    <xacro:property name="link2_to_link3_tran" value="link2_to_link3_tran" />
+    <xacro:property name="link3_to_link4_tran" value="link3_to_link4_tran" />
+    <xacro:property name="link4_to_link5_tran" value="link4_to_link5_tran" />
+    <xacro:property name="link5_to_link6_tran" value="link5_to_link6_tran" />
+    <xacro:property name="link6_to_link7_tran" value="link6_to_link7_tran" />
+    <xacro:property name="link7_to_link8_tran" value="link7_to_link8_tran" />
+    <xacro:property name="base_to_link1_motor" value="base_to_link1_motor" />
+    <xacro:property name="link1_to_link2_motor" value="link1_to_link2_motor" />
+    <xacro:property name="link2_to_link3_motor" value="link2_to_link3_motor" />
+    <xacro:property name="link3_to_link4_motor" value="link3_to_link4_motor" />
+    <xacro:property name="link4_to_link5_motor" value="link4_to_link5_motor" />
+    <xacro:property name="link5_to_link6_motor" value="link5_to_link6_motor" />
+    <xacro:property name="link6_to_link7_motor" value="link6_to_link7_motor" />
+    <xacro:property name="link7_to_link8_motor" value="link7_to_link8_motor" />
+    <!-- Macro to define transmission element -->
+    <xacro:macro name="joint_transmission_macro" params="tran_name motor_name joint_name">
+        <transmission name="${tran_name}">
+            <type>transmission_interface/SimpleTransmission</type>
+            <actuator name="${motor_name}">
+              <mechanicalReduction>1</mechanicalReduction>
+            </actuator>
+            <joint name="${joint_name}">
+              <hardwareInterface>hardware_interface/EffortJointInterface</hardwareInterface>
+            </joint>
+          </transmission>
+    </xacro:macro>
+    <!-- Macro to define ros_control element for joints -->
+    <xacro:macro name="ros_control_joint_macro" params="joint_name">
+        <joint name="${joint_name}">
+            <command_interface name="effort">
+                <param name="min">-200</param>
+                <param name="max">200</param>
+            </command_interface>
+            <state_interface name="effort"/>
+            <state_interface name="position"/>
+            <state_interface name="velocity"/>
+        </joint>
+    </xacro:macro>
+    <!-- Macro to define gazebo link reference element for joints -->
+    <xacro:macro name="gazebo_link_reference_macro" params="link_name gazebo_color_name">
+        <gazebo reference="${link_name}">
+            <material>${gazebo_color_name}</material>
+            <mu1>0.01</mu1>
+            <mu2>0.05</mu2>
+        </gazebo>
+    </xacro:macro>
+    <!-- Gazebo link reference definition with color definition -->
+    <xacro:gazebo_link_reference_macro link_name="${base_link}" gazebo_color_name="Gazebo/Red"/>
+    <xacro:gazebo_link_reference_macro link_name="${link1}" gazebo_color_name="Gazebo/Blue"/>
+    <xacro:gazebo_link_reference_macro link_name="${link2}" gazebo_color_name="Gazebo/Red"/>
+    <xacro:gazebo_link_reference_macro link_name="${link3}" gazebo_color_name="Gazebo/Blue"/>
+    <xacro:gazebo_link_reference_macro link_name="${link4}" gazebo_color_name="Gazebo/Red"/>
+    <xacro:gazebo_link_reference_macro link_name="${link5}" gazebo_color_name="Gazebo/Blue"/>
+    <xacro:gazebo_link_reference_macro link_name="${link6}" gazebo_color_name="Gazebo/Red"/>
+    <xacro:gazebo_link_reference_macro link_name="${link7}" gazebo_color_name="Gazebo/Blue"/>
+    <xacro:gazebo_link_reference_macro link_name="${link8}" gazebo_color_name="Gazebo/Red"/>
+    <ros2_control name="GazeboSystem" type="system">
+    	<hardware>
+            <plugin>gazebo_ros2_control/GazeboSystem</plugin>
+    	</hardware>
+        <xacro:ros_control_joint_macro joint_name="${base_to_link1_Zaxis}"/>
+        <xacro:ros_control_joint_macro joint_name="${link1_to_link2_Xaxis}"/>
+        <xacro:ros_control_joint_macro joint_name="${link2_to_link3_Zaxis}"/>
+        <xacro:ros_control_joint_macro joint_name="${link3_to_link4_Xaxis}"/>
+        <xacro:ros_control_joint_macro joint_name="${link4_to_link5_Zaxis}"/>
+        <xacro:ros_control_joint_macro joint_name="${link5_to_link6_Xaxis}"/>
+        <xacro:ros_control_joint_macro joint_name="${link6_to_link7_Zaxis}"/>
+        <xacro:ros_control_joint_macro joint_name="${link7_to_link8_Xaxis}"/>
+    </ros2_control>
     <gazebo>
-        <!-- plugin to publish the states of the robot joints to generate TF -->
-        <plugin name="gazebo_ros_joint_state_publisher" filename="libgazebo_ros_joint_state_publisher.so">
-            <!-- Update rate in Hertz -->
-            <update_rate>10</update_rate>
-            <!-- Name of joints in the model whose states will be published. -->
-            <joint_name>base_to_link1_Zaxis</joint_name>
-            <joint_name>link1_to_link2_Xaxis</joint_name>
-            <joint_name>link2_to_link3_Zaxis</joint_name>
-            <joint_name>link3_to_link4_Xaxis</joint_name>
-            <joint_name>link4_to_link5_Zaxis</joint_name>
-            <joint_name>link5_to_link6_Xaxis</joint_name>
-            <joint_name>link6_to_link7_Zaxis</joint_name>
-            <joint_name>link7_to_link8_Xaxis</joint_name>
+        <plugin name="gazebo_ros2_control" filename="libgazebo_ros2_control.so">
+        <robot_sim_type>gazebo_ros2_control/GazeboSystem</robot_sim_type>
+        <parameters>$(find snake_robot_description)/config/my_controllers.yaml</parameters>
         </plugin>
     </gazebo>
-    <gazebo>
-        <!-- plugin to set the states of the robot joints -->
-        <plugin name="gazebo_ros_joint_pose_trajectory" filename="libgazebo_ros_joint_pose_trajectory.so">
-            <!-- Update rate in Hz -->
-            <update_rate>2</update_rate>
-        </plugin>
-    </gazebo>
+    <xacro:joint_transmission_macro tran_name="${base_to_link1_tran}" motor_name="${base_to_link1_motor}" joint_name="${base_to_link1_Zaxis}"/>
+    <xacro:joint_transmission_macro tran_name="${link1_to_link2_tran}" motor_name="${link1_to_link2_motor}" joint_name="${link1_to_link2_Xaxis}"/>
+    <xacro:joint_transmission_macro tran_name="${link2_to_link3_tran}" motor_name="${link2_to_link3_motor}" joint_name="${link2_to_link3_Zaxis}"/>
+    <xacro:joint_transmission_macro tran_name="${link3_to_link4_tran}" motor_name="${link3_to_link4_motor}" joint_name="${link3_to_link4_Xaxis}"/>
+    <xacro:joint_transmission_macro tran_name="${link4_to_link5_tran}" motor_name="${link4_to_link5_motor}" joint_name="${link4_to_link5_Zaxis}"/>
+    <xacro:joint_transmission_macro tran_name="${link5_to_link6_tran}" motor_name="${link5_to_link6_motor}" joint_name="${link5_to_link6_Xaxis}"/>
+    <xacro:joint_transmission_macro tran_name="${link6_to_link7_tran}" motor_name="${link6_to_link7_motor}" joint_name="${link6_to_link7_Zaxis}"/>
+    <xacro:joint_transmission_macro tran_name="${link7_to_link8_tran}" motor_name="${link7_to_link8_motor}" joint_name="${link7_to_link8_Xaxis}"/>
 </robot>
