Commit message: still not working

File: snake_ws/install/snake_robot_description/share/snake_robot_description/urdf/snake_camera.xacro (robot description, xacro)
@@ -1,7 +1,8 @@
 <?xml version="1.0"?>
-<robot xmlns:xacro="http://ros.org/wiki/xacro">
+<robot xmlns:xacro="http://ros.org/wiki/xacro" name="snake_robot">
     <xacro:property name="camera_length" value="0.05" />
     <xacro:property name="camera_width" value="0.02" />
     <xacro:property name="camera_height" value="0.05" />
+    <xacro:property name="camera_link" value="camera_link" />
     <!-- link to hold camera -->
     <link name="camera_link">
@@ -20,10 +21,10 @@
     </link>
     <joint name="base_camera_joint" type="fixed">
-        <parent link="base_link" />
-        <child link="camera_link" />
+        <parent link="${link8}" />
+        <child link="${camera_link}"  />
         <!-- the RPY is NOT 000 to make sure camera does not see inside ground but is over the surface -->
-        <origin xyz="0 -${(pipelen + camera_width) / 2} ${piperdius}" rpy="0 -${pi / 16.0} -${pi / 2.0}" />
+        <origin xyz="0 -${(pipelen + camera_width) / 2} ${piperdius}" rpy="0 -${pi / 16.0} ${pi / 2.0}" />
     </joint>
-    <!-- camera plugin for gazebo -->
+    <!-- camera plugin and link reference for gazebo -->
     <gazebo reference="camera_link">
         <material>Gazebo/Red</material>

File: snake_ws/install/snake_robot_description/share/snake_robot_description/urdf/snake_common_properties.xacro (robot description, xacro)
@@ -1,4 +1,5 @@
 <?xml version="1.0"?>
-<robot xmlns:xacro="http://ros.org/wiki/xacro">
+<robot xmlns:xacro="http://ros.org/wiki/xacro" name="snake_robot">
+    <xacro:property name="robot_name" value="snake_robot" />
     <!-- Define a color materials with RGBA color values -->
     <material name="blue">

File: snake_ws/install/snake_robot_description/share/snake_robot_description/urdf/snake_components.xacro (robot description, xacro)
@@ -1,7 +1,30 @@
 <?xml version="1.0"?>
-<robot xmlns:xacro="http://ros.org/wiki/xacro">
+<robot xmlns:xacro="http://ros.org/wiki/xacro" name="snake_robot">
+    <!-- Property to define link names -->
+    <xacro:property name="base_link" value="base_link" />
+    <xacro:property name="link1" value="link1" />
+    <xacro:property name="link2" value="link2" />
+    <xacro:property name="link3" value="link3" />
+    <xacro:property name="link4" value="link4" />
+    <xacro:property name="link5" value="link5" />
+    <xacro:property name="link6" value="link6" />
+    <xacro:property name="link7" value="link7" />
+    <xacro:property name="link8" value="link8" />
+    <!-- Property to define joint names -->
+    <xacro:property name="base_to_link1_Zaxis_joint" value="basetolink1_Z" />
+    <xacro:property name="link1_to_link2_Xaxis_joint" value="link1to2_X" />
+    <xacro:property name="link2_to_link3_Zaxis_joint" value="link2to3_Z" />
+    <xacro:property name="link3_to_link4_Xaxis_joint" value="link3to4_X" />
+    <xacro:property name="link4_to_link5_Zaxis_joint" value="link4to5_Z" />
+    <xacro:property name="link5_to_link6_Xaxis_joint" value="link5to6_X" />
+    <xacro:property name="link6_to_link7_Zaxis_joint" value="link6to7_Z" />
+    <xacro:property name="link7_to_link8_Xaxis_joint" value="link7to8_X" />
     <!-- Define variables for reuse -->
     <xacro:property name="piperdius" value="0.1" />
     <xacro:property name="pipelen" value="0.4" />
+    <odometry_frame>odom</odometry_frame>
+    <publish_odom>true</publish_odom>
+    <publish_odom_tf>true</publish_odom_tf>
+    <publish_joint_tf></publish_joint_tf>
     <!-- Define a macro to create a link with visual, collision, and inertia properties -->
     <xacro:macro name="link_macro" params="name x_origin y_origin z_origin color">
@@ -26,5 +49,5 @@
     </xacro:macro>
     <!-- Define a macro to create a revolute joint along the Z-axis between two links -->
-    <xacro:macro name="link_to_link_Zaxis_macro" params="name x_origin y_origin z_origin parent child">
+    <xacro:macro name="joint_Zaxis_macro" params="name x_origin y_origin z_origin parent child">
         <joint name="${name}" type="revolute">
             <axis xyz="0 0 1"/>
@@ -37,5 +60,5 @@
     </xacro:macro>
     <!-- Define a macro to create a revolute joint along the X-axis between two links -->
-    <xacro:macro name="link_to_link_Xaxis_macro" params="name x_origin y_origin z_origin parent child">
+    <xacro:macro name="joint_Xaxis_macro" params="name x_origin y_origin z_origin parent child">
         <joint name="${name}" type="revolute">
             <axis xyz="1 0 0"/>
@@ -48,22 +71,41 @@
         </joint>
     </xacro:macro>
+    <xacro:macro name="default_transmission" params="jointname">
+        <transmission name="${jointname}_trnsmsn">
+            <plugin>transmission_interface/SimpleTransmission</plugin>
+            <actuator name="${jointname}_motor">
+                <mechanicalReduction>1.0</mechanicalReduction>
+            </actuator>
+            <joint name="${jointname}">
+                <hardwareInterface>hardware_interface/EffortJointInterface</hardwareInterface>
+            </joint>
+        </transmission>
+    </xacro:macro>
     <!-- Create the base link with red color -->
-    <xacro:link_macro name="base_link" x_origin="0" y_origin="0" z_origin="${piperdius}" color="red"/>
+    <xacro:link_macro name="${base_link}" x_origin="0" y_origin="0" z_origin="${piperdius}" color="red"/>
     <!-- Create links, joints, and set their positions and colors -->
-    <xacro:link_to_link_Zaxis_macro name="base_to_link1_Zaxis" x_origin="0" y_origin="${pipelen / 2}" z_origin="${piperdius}" parent="base_link" child="link1"/>
-    <xacro:link_macro name="link1" x_origin="0" y_origin="${pipelen / 2}" z_origin="0" color="blue"/>
-    <xacro:link_to_link_Xaxis_macro name="link1_to_link2_Xaxis" x_origin="0" y_origin="${pipelen}" z_origin="0" parent="link1" child="link2"/>
-    <xacro:link_macro name="link2" x_origin="0" y_origin="${pipelen / 2}" z_origin="0" color="red"/>
-    <xacro:link_to_link_Zaxis_macro name="link2_to_link3_Zaxis" x_origin="0" y_origin="${pipelen}" z_origin="0" parent="link2" child="link3"/>
-    <xacro:link_macro name="link3" x_origin="0" y_origin="${pipelen / 2}" z_origin="0" color="blue"/>
-    <xacro:link_to_link_Xaxis_macro name="link3_to_link4_Xaxis" x_origin="0" y_origin="${pipelen}" z_origin="0" parent="link3" child="link4"/>
-    <xacro:link_macro name="link4" x_origin="0" y_origin="${pipelen / 2}" z_origin="0" color="red"/>
-    <xacro:link_to_link_Zaxis_macro name="link4_to_link5_Zaxis" x_origin="0" y_origin="${pipelen}" z_origin="0" parent="link4" child="link5"/>
-    <xacro:link_macro name="link5" x_origin="0" y_origin="${pipelen / 2}" z_origin="0" color="blue"/>
-    <xacro:link_to_link_Xaxis_macro name="link5_to_link6_Xaxis" x_origin="0" y_origin="${pipelen}" z_origin="0" parent="link5" child="link6"/>
-    <xacro:link_macro name="link6" x_origin="0" y_origin="${pipelen / 2}" z_origin="0" color="red"/>
-    <xacro:link_to_link_Zaxis_macro name="link6_to_link7_Zaxis" x_origin="0" y_origin="${pipelen}" z_origin="0" parent="link6" child="link7"/>
-    <xacro:link_macro name="link7" x_origin="0" y_origin="${pipelen / 2}" z_origin="0" color="blue"/>
-    <xacro:link_to_link_Xaxis_macro name="link7_to_link8_Xaxis" x_origin="0" y_origin="${pipelen}" z_origin="0" parent="link7" child="link8"/>
-    <xacro:link_macro name="link8" x_origin="0" y_origin="${pipelen / 2}" z_origin="0" color="red"/>
+    <xacro:joint_Zaxis_macro name="${base_to_link1_Zaxis_joint}" x_origin="0" y_origin="${pipelen / 2}" z_origin="${piperdius}" parent="${base_link}" child="${link1}"/>
+    <xacro:link_macro name="${link1}" x_origin="0" y_origin="${pipelen / 2}" z_origin="0" color="blue"/>
+    <xacro:default_transmission jointname="${base_to_link1_Zaxis_joint}"/>
+    <xacro:joint_Xaxis_macro name="${link1_to_link2_Xaxis_joint}" x_origin="0" y_origin="${pipelen}" z_origin="0" parent="${link1}" child="${link2}"/>
+    <xacro:link_macro name="${link2}" x_origin="0" y_origin="${pipelen / 2}" z_origin="0" color="red"/>
+    <xacro:default_transmission jointname="${link1_to_link2_Xaxis_joint}"/>
+    <xacro:joint_Zaxis_macro name="${link2_to_link3_Zaxis_joint}" x_origin="0" y_origin="${pipelen}" z_origin="0" parent="${link2}" child="${link3}"/>
+    <xacro:link_macro name="${link3}" x_origin="0" y_origin="${pipelen / 2}" z_origin="0" color="blue"/>
+    <xacro:default_transmission jointname="${link2_to_link3_Zaxis_joint}"/>
+    <xacro:joint_Xaxis_macro name="${link3_to_link4_Xaxis_joint}" x_origin="0" y_origin="${pipelen}" z_origin="0" parent="${link3}" child="${link4}"/>
+    <xacro:link_macro name="${link4}" x_origin="0" y_origin="${pipelen / 2}" z_origin="0" color="red"/>
+    <xacro:default_transmission jointname="${link3_to_link4_Xaxis_joint}"/>
+    <xacro:joint_Zaxis_macro name="${link4_to_link5_Zaxis_joint}" x_origin="0" y_origin="${pipelen}" z_origin="0" parent="${link4}" child="${link5}"/>
+    <xacro:link_macro name="${link5}" x_origin="0" y_origin="${pipelen / 2}" z_origin="0" color="blue"/>
+    <xacro:default_transmission jointname="${link4_to_link5_Zaxis_joint}"/>
+    <xacro:joint_Xaxis_macro name="${link5_to_link6_Xaxis_joint}" x_origin="0" y_origin="${pipelen}" z_origin="0" parent="${link5}" child="${link6}"/>
+    <xacro:link_macro name="${link6}" x_origin="0" y_origin="${pipelen / 2}" z_origin="0" color="red"/>
+    <xacro:default_transmission jointname="${link5_to_link6_Xaxis_joint}"/>
+    <xacro:joint_Zaxis_macro name="${link6_to_link7_Zaxis_joint}" x_origin="0" y_origin="${pipelen}" z_origin="0" parent="${link6}" child="${link7}"/>
+    <xacro:link_macro name="${link7}" x_origin="0" y_origin="${pipelen / 2}" z_origin="0" color="blue"/>
+    <xacro:default_transmission jointname="${link6_to_link7_Zaxis_joint}"/>
+    <xacro:joint_Xaxis_macro name="${link7_to_link8_Xaxis_joint}" x_origin="0" y_origin="${pipelen}" z_origin="0" parent="${link7}" child="${link8}"/>
+    <xacro:link_macro name="${link8}" x_origin="0" y_origin="${pipelen / 2}" z_origin="0" color="red"/>
+    <xacro:default_transmission jointname="${link7_to_link8_Xaxis_joint}"/>
 </robot>

File: snake_ws/install/snake_robot_description/share/snake_robot_description/urdf/snake_components_gazebo.xacro (robot description, xacro)
@@ -1,53 +1,54 @@
 <?xml version="1.0"?>
-<robot xmlns:xacro="http://ros.org/wiki/xacro">
-    <gazebo reference="base_link">
+<robot xmlns:xacro="http://ros.org/wiki/xacro" name="snake_robot">
+    <gazebo reference="${base_link}">
         <material>Gazebo/Red</material>
+        <mu1>0.01</mu1>
+        <mu2>0.05</mu2>
     </gazebo>
-    <gazebo reference="link1">
+    <gazebo reference="${link1}">
         <material>Gazebo/Blue</material>
+        <mu1>0.01</mu1>
+        <mu2>0.05</mu2>
     </gazebo>
-    <gazebo reference="link2">
+    <gazebo reference="${link2}">
         <material>Gazebo/Red</material>
+        <mu1>0.01</mu1>
+        <mu2>0.05</mu2>
     </gazebo>
-    <gazebo reference="link3">
+    <gazebo reference="${link3}">
         <material>Gazebo/Blue</material>
+        <mu1>0.01</mu1>
+        <mu2>0.05</mu2>
     </gazebo>
-    <gazebo reference="link4">
+    <gazebo reference="${link4}">
         <material>Gazebo/Red</material>
+        <mu1>0.01</mu1>
+        <mu2>0.05</mu2>
     </gazebo>
-    <gazebo reference="link5">
+    <gazebo reference="${link5}">
         <material>Gazebo/Blue</material>
+        <mu1>0.01</mu1>
+        <mu2>0.05</mu2>
     </gazebo>
-    <gazebo reference="link6">
+    <gazebo reference="${link6}">
         <material>Gazebo/Red</material>
+        <mu1>0.01</mu1>
+        <mu2>0.05</mu2>
     </gazebo>
-    <gazebo reference="link7">
+    <gazebo reference="${link7}">
         <material>Gazebo/Blue</material>
+        <mu1>0.01</mu1>
+        <mu2>0.05</mu2>
     </gazebo>
-    <gazebo reference="link8">
+    <gazebo reference="${link8}">
         <material>Gazebo/Red</material>
+        <mu1>0.01</mu1>
+        <mu2>0.05</mu2>
     </gazebo>
-    <!-- Plugin introduced from https://github.com/ros-simulation/gazebo_ros_pkgs/blob/ros2/gazebo_plugins/include/gazebo_plugins/gazebo_ros_joint_state_publisher.hpp -->
+    <!-- code for GAZEBO_ROS_CONTROL -->
     <gazebo>
-        <!-- plugin to publish the states of the robot joints to generate TF -->
-        <plugin name="gazebo_ros_joint_state_publisher" filename="libgazebo_ros_joint_state_publisher.so">
-            <!-- Update rate in Hertz -->
-            <update_rate>10</update_rate>
-            <!-- Name of joints in the model whose states will be published. -->
-            <joint_name>base_to_link1_Zaxis</joint_name>
-            <joint_name>link1_to_link2_Xaxis</joint_name>
-            <joint_name>link2_to_link3_Zaxis</joint_name>
-            <joint_name>link3_to_link4_Xaxis</joint_name>
-            <joint_name>link4_to_link5_Zaxis</joint_name>
-            <joint_name>link5_to_link6_Xaxis</joint_name>
-            <joint_name>link6_to_link7_Zaxis</joint_name>
-            <joint_name>link7_to_link8_Xaxis</joint_name>
-        </plugin>
-    </gazebo>
-    <gazebo>
-        <!-- plugin to set the states of the robot joints -->
-        <plugin name="gazebo_ros_joint_pose_trajectory" filename="libgazebo_ros_joint_pose_trajectory.so">
-            <!-- Update rate in Hz -->
-            <update_rate>2</update_rate>
+        <plugin name="gazebo_ros2_control" filename="libgazebo_ros2_control.so" >
+            <robot_sim_type>gazebo_ros2_control/GazeboSystem</robot_sim_type>
+            <parameters>$(find snake_robot_description)/config/snake_controllers.yaml</parameters>
         </plugin>
     </gazebo>

File: snake_ws/install/snake_robot_description/share/snake_robot_description/urdf/snake_urdf.xacro (robot description, xacro)
@@ -1,7 +1,8 @@
 <?xml version="1.0"?>
-<robot name="snake robot" xmlns:xacro="http://ros.org/wiki/xacro">
-    <xacro:include filename="snake_common_properties.xacro" />
-    <xacro:include filename="snake_components.xacro" />
-    <xacro:include filename="snake_components_gazebo.xacro" />
-    <xacro:include filename="snake_camera.xacro" />
+<robot name="snake_robot" xmlns:xacro="http://ros.org/wiki/xacro">
+    <xacro:include filename="$(find snake_robot_description)/urdf/snake_common_properties.xacro" />
+    <xacro:include filename="$(find snake_robot_description)/urdf/snake_components.xacro" />
+    <xacro:include filename="$(find snake_robot_description)/urdf/snake_camera.xacro" />
+    <xacro:include filename="$(find snake_robot_description)/urdf/snake_components_gazebo.xacro" />
+    <xacro:include filename="$(find snake_robot_description)/urdf/snake_ros2_control.xacro" />
 </robot>
