Commit message: still not working

File: snake_ws/src/snake_robot_description/urdf/snake_ros2_control.xacro (robot description, xacro)
@@ -1,11 +1,13 @@
 <?xml version="1.0" encoding="UTF-8"?>
-<robot name="${robot_name}" xmlns:xacro="http://ros.org/wiki/xacro">
+<robot name="snake_robot" xmlns:xacro="http://ros.org/wiki/xacro">
     <xacro:macro name="ros2Control_joint_section" params="jointname">
         <joint name="${jointname}">
-            <command_interface name="position">
+            <command_interface name="effort">
                 <param name="min">-${pi / 2.0}</param>
                 <param name="max">${pi / 2.0}</param>
             </command_interface>
-            <state_interface name="position" />
+            <state_interface name="effort"/>
+            <state_interface name="position"/>
+            <state_interface name="velocity"/>
         </joint>
     </xacro:macro>

File: snake_ws/src/snake_robot_description/urdf/snake_urdf.xacro (robot description, xacro)
@@ -1,8 +1,8 @@
 <?xml version="1.0"?>
-<robot name="${robot_name}" xmlns:xacro="http://ros.org/wiki/xacro">
+<robot name="snake_robot" xmlns:xacro="http://ros.org/wiki/xacro">
     <xacro:include filename="$(find snake_robot_description)/urdf/snake_common_properties.xacro" />
+    <xacro:include filename="$(find snake_robot_description)/urdf/snake_components.xacro" />
+    <xacro:include filename="$(find snake_robot_description)/urdf/snake_camera.xacro" />
+    <xacro:include filename="$(find snake_robot_description)/urdf/snake_components_gazebo.xacro" />
     <xacro:include filename="$(find snake_robot_description)/urdf/snake_ros2_control.xacro" />
-    <xacro:include filename="snake_components.xacro" />
-    <xacro:include filename="snake_components_gazebo.xacro" />
-    <xacro:include filename="snake_camera.xacro" />
 </robot>
