Commit message: working with tutorial

File: snake_ws/src/snake_robot_description/urdf/scratch.xacro (robot description, xacro)
@@ -15,12 +15,12 @@
     <xacro:property name="link8" value="link8" />
     <!-- Property to define joint names -->
-    <xacro:property name="base_to_link1_Zaxis_joint" value="basetolink1_Z" />
-    <xacro:property name="link1_to_link2_Xaxis_joint" value="link1to2_X" />
-    <xacro:property name="link2_to_link3_Zaxis_joint" value="link23_Z" />
-    <xacro:property name="link3_to_link4_Xaxis_joint" value="link34_X" />
-    <xacro:property name="link4_to_link5_Zaxis_joint" value="link45_Z" />
-    <xacro:property name="link5_to_link6_Xaxis_joint" value="link56_X" />
-    <xacro:property name="link6_to_link7_Zaxis_joint" value="link67_Z" />
-    <xacro:property name="link7_to_link8_Xaxis_joint" value="link78_X" />
+    <xacro:property name="base_to_link1_Zaxis" value="base_to_link1_Zaxis" />
+    <xacro:property name="link1_to_link2_Xaxis" value="link1_to_link2_Xaxis" />
+    <xacro:property name="link2_to_link3_Zaxis" value="link2_to_link3_Zaxis" />
+    <xacro:property name="link3_to_link4_Xaxis" value="link3_to_link4_Xaxis" />
+    <xacro:property name="link4_to_link5_Zaxis" value="link4_to_link5_Zaxis" />
+    <xacro:property name="link5_to_link6_Xaxis" value="link5_to_link6_Xaxis" />
+    <xacro:property name="link6_to_link7_Zaxis" value="link6_to_link7_Zaxis" />
+    <xacro:property name="link7_to_link8_Xaxis" value="link7_to_link8_Xaxis" />
     <!-- Define a macro to create a link with visual, collision, and inertia properties -->
     <xacro:macro name="link_macro" params="name x_origin y_origin z_origin color">
@@ -45,5 +45,5 @@
     </xacro:macro>
     <!-- Define a macro to create a revolute joint along the Z-axis between two links -->
-    <xacro:macro name="joint_Zaxis_macro" params="name x_origin y_origin z_origin parent child">
+    <xacro:macro name="link_to_link_Zaxis_joint_macro" params="name x_origin y_origin z_origin parent child">
         <joint name="${name}" type="revolute">
             <axis xyz="0 0 1"/>
@@ -56,5 +56,5 @@
     </xacro:macro>
     <!-- Define a macro to create a revolute joint along the X-axis between two links -->
-    <xacro:macro name="joint_Xaxis_macro" params="name x_origin y_origin z_origin parent child">
+    <xacro:macro name="link_to_link_Xaxis_joint_macro" params="name x_origin y_origin z_origin parent child">
         <joint name="${name}" type="revolute">
             <axis xyz="1 0 0"/>
@@ -67,39 +67,22 @@
         </joint>
     </xacro:macro>
-    <xacro:macro name="default_transmission" params="jointname">
-        <transmission name="${jointname}_trnsmsn">
-            <plugin>transmission_interface/SimpleTransmission</plugin>
-            <actuator name="${jointname}_motor" role="actuator1" />
-            <joint name="${jointname}" role="joint1">
-                <mechanicalReduction>1.0</mechanicalReduction>
-            </joint>
-        </transmission>
-    </xacro:macro>
     <!-- Create the base link with red color -->
     <xacro:link_macro name="${base_link}" x_origin="0" y_origin="0" z_origin="${piperdius}" color="red"/>
     <!-- Create links, joints, and set their positions and colors -->
-    <xacro:link_to_link_Zaxis_joint_macro name="${base_to_link1_Zaxis_joint}" x_origin="0" y_origin="${pipelen / 2}" z_origin="${piperdius}" parent="${base_link}" child="${link1}"/>
+    <xacro:link_to_link_Zaxis_joint_macro name="${base_to_link1_Zaxis}" x_origin="0" y_origin="${pipelen / 2}" z_origin="${piperdius}" parent="${base_link}" child="${link1}"/>
     <xacro:link_macro name="${link1}" x_origin="0" y_origin="${pipelen / 2}" z_origin="0" color="blue"/>
-    <xacro:default_transmission jointname="${base_to_link1_Zaxis_joint}"/>
-    <xacro:link_to_link_Xaxis_joint_macro name="${link1_to_link2_Xaxis_joint}" x_origin="0" y_origin="${pipelen}" z_origin="0" parent="${link1}" child="${link2}"/>
+    <xacro:link_to_link_Xaxis_joint_macro name="${link1_to_link2_Xaxis}" x_origin="0" y_origin="${pipelen}" z_origin="0" parent="${link1}" child="${link2}"/>
     <xacro:link_macro name="${link2}" x_origin="0" y_origin="${pipelen / 2}" z_origin="0" color="red"/>
-    <xacro:default_transmission jointname="${link1_to_link2_Xaxis_joint}"/>
-    <xacro:link_to_link_Zaxis_joint_macro name="${link2_to_link3_Zaxis_joint}" x_origin="0" y_origin="${pipelen}" z_origin="0" parent="${link2}" child="${link3}"/>
+    <xacro:link_to_link_Zaxis_joint_macro name="${link2_to_link3_Zaxis}" x_origin="0" y_origin="${pipelen}" z_origin="0" parent="${link2}" child="${link3}"/>
     <xacro:link_macro name="${link3}" x_origin="0" y_origin="${pipelen / 2}" z_origin="0" color="blue"/>
-    <xacro:default_transmission jointname="${link2_to_link3_Zaxis_joint}"/>
-    <xacro:link_to_link_Xaxis_joint_macro name="${link3_to_link4_Xaxis_joint}" x_origin="0" y_origin="${pipelen}" z_origin="0" parent="${link3}" child="${link4}"/>
+    <xacro:link_to_link_Xaxis_joint_macro name="${link3_to_link4_Xaxis}" x_origin="0" y_origin="${pipelen}" z_origin="0" parent="${link3}" child="${link4}"/>
     <xacro:link_macro name="${link4}" x_origin="0" y_origin="${pipelen / 2}" z_origin="0" color="red"/>
-    <xacro:default_transmission jointname="${link3_to_link4_Xaxis_joint}"/>
-    <xacro:link_to_link_Zaxis_joint_macro name="${link4_to_link5_Zaxis_joint}" x_origin="0" y_origin="${pipelen}" z_origin="0" parent="${link4}" child="${link5}"/>
+    <xacro:link_to_link_Zaxis_joint_macro name="${link4_to_link5_Zaxis}" x_origin="0" y_origin="${pipelen}" z_origin="0" parent="${link4}" child="${link5}"/>
     <xacro:link_macro name="${link5}" x_origin="0" y_origin="${pipelen / 2}" z_origin="0" color="blue"/>
-    <xacro:default_transmission jointname="${link4_to_link5_Zaxis_joint}"/>
-    <xacro:link_to_link_Xaxis_joint_macro name="${link5_to_link6_Xaxis_joint}" x_origin="0" y_origin="${pipelen}" z_origin="0" parent="${link5}" child="${link6}"/>
+    <xacro:link_to_link_Xaxis_joint_macro name="${link5_to_link6_Xaxis}" x_origin="0" y_origin="${pipelen}" z_origin="0" parent="${link5}" child="${link6}"/>
     <xacro:link_macro name="${link6}" x_origin="0" y_origin="${pipelen / 2}" z_origin="0" color="red"/>
-    <xacro:default_transmission jointname="${link5_to_link6_Xaxis_joint}"/>
-    <xacro:link_to_link_Zaxis_joint_macro name="${link6_to_link7_Zaxis_joint}" x_origin="0" y_origin="${pipelen}" z_origin="0" parent="${link6}" child="${link7}"/>
+    <xacro:link_to_link_Zaxis_joint_macro name="${link6_to_link7_Zaxis}" x_origin="0" y_origin="${pipelen}" z_origin="0" parent="${link6}" child="${link7}"/>
     <xacro:link_macro name="${link7}" x_origin="0" y_origin="${pipelen / 2}" z_origin="0" color="blue"/>
-    <xacro:default_transmission jointname="${link6_to_link7_Zaxis_joint}"/>
-    <xacro:link_to_link_Xaxis_joint_macro name="${link7_to_link8_Xaxis_joint}" x_origin="0" y_origin="${pipelen}" z_origin="0" parent="${link7}" child="${link8}"/>
+    <xacro:link_to_link_Xaxis_joint_macro name="${link7_to_link8_Xaxis}" x_origin="0" y_origin="${pipelen}" z_origin="0" parent="${link7}" child="${link8}"/>
     <xacro:link_macro name="${link8}" x_origin="0" y_origin="${pipelen / 2}" z_origin="0" color="red"/>
-    <xacro:default_transmission jointname="${link7_to_link8_Xaxis_joint}"/>
 </robot>

File: snake_ws/src/snake_robot_description/urdf/snake_camera.xacro (robot description, xacro)
@@ -1,4 +1,4 @@
 <?xml version="1.0"?>
-<robot xmlns:xacro="http://ros.org/wiki/xacro">
+<robot xmlns:xacro="http://ros.org/wiki/xacro" name="${robot_name}">
     <xacro:property name="camera_length" value="0.05" />
     <xacro:property name="camera_width" value="0.02" />

File: snake_ws/src/snake_robot_description/urdf/snake_common_properties.xacro (robot description, xacro)
@@ -1,4 +1,5 @@
 <?xml version="1.0"?>
-<robot xmlns:xacro="http://ros.org/wiki/xacro">
+<robot xmlns:xacro="http://ros.org/wiki/xacro" name="${robot_name}">
+    <xacro:property name="robot_name" value="snake_robot" />
     <!-- Define a color materials with RGBA color values -->
     <material name="blue">

File: snake_ws/src/snake_robot_description/urdf/snake_components_gazebo.xacro (robot description, xacro)
@@ -1,4 +1,4 @@
 <?xml version="1.0"?>
-<robot xmlns:xacro="http://ros.org/wiki/xacro">
+<robot xmlns:xacro="http://ros.org/wiki/xacro" name="${robot_name}">
     <gazebo reference="base_link">
         <material>Gazebo/Red</material>
@@ -52,3 +52,11 @@
         </plugin>
     </gazebo>
+    <!-- code for ROS_CONTROL -->
+    <gazebo>
+        <plugin filename="libgazebo_ros2_control.so" name="gazebo_ros2_control">
+            <robot_param>robot_description</robot_param>
+            <robot_param_node>robot_state_publisher</robot_param_node>
+            <parameters></parameters>
+        </plugin>
+    </gazebo>
 </robot>

File: snake_ws/src/snake_robot_description/urdf/snake_urdf.xacro (robot description, xacro)
@@ -1,5 +1,6 @@
 <?xml version="1.0"?>
-<robot name="snake robot" xmlns:xacro="http://ros.org/wiki/xacro">
-    <xacro:include filename="snake_common_properties.xacro" />
+<robot name="${robot_name}" xmlns:xacro="http://ros.org/wiki/xacro">
+    <xacro:include filename="$(find snake_robot_description)/urdf/snake_common_properties.xacro" />
+    <xacro:include filename="$(find snake_robot_description)/urdf/snake_ros2_control.xacro" />
     <xacro:include filename="snake_components.xacro" />
     <xacro:include filename="snake_components_gazebo.xacro" />
